File: KiCad Files/3374_VCO.kicad_pcb (KiCad board)
At the start: 4 copper layers, 11.2 x 25.4 mm, 70 parts, among them J1 FLIP PINS, J2 FLIP PINS, Q1 DMMT3906W, Q10 DMMT3906W, Q11 DMMT3904W, Q12 DMMT3906W, Q13 DMMT3904W, Q14 DMMT3904W, Q15 DMMT3904W, Q2 MUN5314DW1, Q3 DMMT3906W, Q4 DMMT3904W, Q5 DMMT3906W, Q6 DMMT3904W, Q7 DMMT3906W, Q8 DMMT3906W, Q9 DMMT3906W, U1 DG636E, U2 DG636E, U3 TL074H, U4 AP7370-50FDC, U5 TLV9032, U6 TL074H, U7 TMP6131DECR

Commit message: Updated to Rev 1
Parts:
- removed the C10 at (114.1, 46.7)
- removed the C11 at (114.1, 49.2)
- removed the C12 at (106.7, 49.8)
- removed the C13 at (114.3, 51.8)
- removed D1: BAW56DW, Package_TO_SOT_SMD:SOT-363_SC-70-6
- removed the Q1 at (111.8, 47.9)
- removed the Q3 at (111.8, 50.9)
- removed the Q8 at (111.8, 47.9)
- removed the Q9 at (109.1, 47.9)
- removed the R10 at (114.3, 42.2)
- removed the R17 at (106.7, 49.2)
- removed the R26 at (112.3, 43.9)
- removed the R4 at (113.0, 38.7)
- removed the R8 at (114.3, 41.6)
- added R1: 432K, Resistor_SMD:R_0201_0603Metric, F.Cu at (106.3, 34.3)
- added R11: 10k, Resistor_SMD:R_0201_0603Metric, F.Cu at (114.3, 44.1)
- added R13: 10k, Resistor_SMD:R_0201_0603Metric, F.Cu at (114.3, 44.8)
- added R15: 3.32k, Resistor_SMD:R_0201_0603Metric, F.Cu at (108.3, 46.3)
- added R18: 10k, Resistor_SMD:R_0201_0603Metric, F.Cu at (114.0, 47.3)
- added R2: 432K, Resistor_SMD:R_0201_0603Metric, F.Cu at (114.3, 39.1)
- added R27: 3.32k, Resistor_SMD:R_0201_0603Metric, B.Cu at (112.5, 46.3)
- C1: renamed from C16; value 0.1u -> 100n; moved to F.Cu
- C10: renamed from C9; value 100p -> 680p
- C11: renamed from C14; value 0.1u -> 100n
- C12: renamed from C15; value 0.1u -> 100n
- C14: renamed from C18; value 100p -> 680p
- C15: renamed from C19; value 0.1u -> 100n
- C16: renamed from C20; value 0.1u -> 100n
- C2: renamed from C1; value 0.1u -> 100n
- C3: renamed from C5; value 0.1u -> 100n
- C4: value 0.001u -> 680p
- C5: renamed from C3; value 0.1u -> 100n
- C6: value 0.1u -> 100n
- C7: renamed from C2; value 0.001u -> 680p
- C8: renamed from C7; value 0.1u -> 100n
- C9: renamed from C8; value 0.1u -> 100n
- R16: value 0 -> 4.99k
- R20: renamed from R19; value 1.02Meg -> 432K
- R21: renamed from R20; value 1.02Meg -> 432K
- R23: renamed from R22; footprint Resistor_SMD:R_0402_1005Metric -> Resistor_SMD:R_0201_0603Metric
- R24: renamed from R6; value 422 -> 365; moved to B.Cu
- R3: renamed from R1; value 422 -> 365
- U1, U2: value DG636E -> DG4053E
- moved R14 6.87 mm to (107.7, 46.0)
- moved C7 5.28 mm to (114.3, 39.7)
- moved R17 4.60 mm to (106.7, 47.0), turned to 180 degrees
- moved C5 4.36 mm to (108.7, 38.4), turned to 180 degrees
- moved R3 4.03 mm to (109.2, 40.3), turned to 180 degrees
- moved R6 3.15 mm to (107.0, 41.6)
- moved C3 2.95 mm to (112.5, 34.0), turned to 0 degrees
- moved C6 2.81 mm to (111.7, 38.6), turned to 180 degrees
- moved C8 2.55 mm to (108.0, 43.5)
- moved R12 2.55 mm to (106.7, 44.8)
- moved R10 2.55 mm to (106.7, 44.1)
- moved R9 2.54 mm to (114.1, 42.2)
- moved R7 2.54 mm to (114.1, 41.6)
- moved C10 2.40 mm to (113.0, 45.1)
- moved C14 2.40 mm to (108.6, 46.3)
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- renumbered C17 to C13, Q2 to Q1, Q14 to Q10, Q15 to Q11, Q4 to Q2, Q5 to Q3, Q6 to Q4, Q7 to Q5, Q10 to Q6, Q11 to Q7, Q12 to Q8, Q13 to Q9, R7 to R10, R9 to R12, R5 to R14, R11 to R17, R18 to R19, R21 to R22, R24 to R25, R25 to R26, R2 to R4, R3 to R5, R14 to R6, R13 to R7, R12 to R8, R15 to R9
Connections:
- C7 pad 1: Net-(C2-Pad1) -> Net-(C7-Pad1)
- Q1 pad 6: Net-(D1D-K) -> CF_A
- Q2 pad 4: -5V -> /VCO A/SHIFTED_TRI_A
- Q2 pad 5: -5V -> /VCO A/SHIFTED_TRI_A
- Q3 pad 4: Net-(Q3A-B1) (its old number) -> +12V
- Q3 pad 5: Net-(Q3A-B1) (its old number) -> +12V
- Q4 pad 1: Net-(Q6A-B1) (its old number) -> Net-(Q4A-B1)
- Q4 pad 2: Net-(Q6A-B1) (its old number) -> Net-(Q4A-B1)
- Q4 pad 3: Net-(Q6A-B1) (its old number) -> Net-(Q4A-B1)
- Q4 pad 6: Net-(D1D-K) -> CF_A
- Q5 pad 6: Net-(Q6A-B1) (its old number) -> Net-(Q5B-C2)
- Q6 pad 4: Net-(Q10A-E1) (its old number) -> +12V
- Q6 pad 5: Net-(Q10A-E1) (its old number) -> +12V
- Q7 pad 4: -5V -> /VCO B/SHIFTED_TRI_B
- Q7 pad 5: -5V -> /VCO B/SHIFTED_TRI_B
- Q8 pad 6: Net-(Q12B-C2) -> Net-(Q8B-C2)
- Q9 pad 1: Net-(Q12B-C2) -> Net-(Q9A-B1)
- Q9 pad 2: Net-(Q12B-C2) -> Net-(Q9A-B1)
- Q9 pad 3: Net-(Q12B-C2) -> Net-(Q9A-B1)
- Q9 pad 6: Net-(D1B-K) -> CF_B
- R12 pad 2: +5V -> TRIANGLE_A
- R14 pad 2: Net-(R5-Pad2) -> GND
- R16 pad 1: Net-(D1B-K) -> Net-(U6D--)
- R16 pad 2: CF_B -> GND
- R17 pad 1: Net-(D1C-K) -> Net-(U3D--)
- R17 pad 2: Net-(U3D--) -> +5V
- R24 pad 2: Net-(C2-Pad1) -> Net-(C7-Pad1)
- U1 pad 1: +5V -> Net-(Q4A-B1)
- U1 pad 11: +5V -> GND
- U1 pad 12: GND -> Net-(U5A--)
- U1 pad 13: Net-(R5-Pad2) -> Net-(U3C-+)
- U1 pad 14: unconnected-(U1C-NC-Pad14) -> +5V
- U1 pad 15: unconnected-(U1C-NC-Pad15) -> VTH_A
- U1 pad 16: Net-(R5-Pad2) -> Net-(C4-Pad1)
- U1 pad 2: -5V -> Net-(Q5B-C2)
- U1 pad 3: Net-(C4-Pad1) -> CF_A
- U1 pad 4: VTH_A -> GND
- U1 pad 5: Net-(U3C-+) -> -5V
- U1 pad 6: unconnected-(U1C-NC-Pad6) -> GND
- U1 pad 7: unconnected-(U1C-NC-Pad7) -> /VCO A/SQUARE_A
- U1 pad 8: Net-(U5B--) -> /VCO A/SQUARE_A
- U1 pad 9: GND -> /VCO A/SQUARE_A
- U2 pad 1: +5V -> Net-(Q9A-B1)
- U2 pad 11: +5V -> GND
- U2 pad 12: GND -> Net-(U5B--)
- U2 pad 13: Net-(R4-Pad1) -> Net-(U6C-+)
- U2 pad 14: unconnected-(U2C-NC-Pad14) -> +5V
- U2 pad 15: unconnected-(U2C-NC-Pad15) -> VTH_B
- U2 pad 16: Net-(R4-Pad1) -> Net-(C7-Pad1)
- U2 pad 2: -5V -> Net-(Q8B-C2)
- U2 pad 3: Net-(C2-Pad1) -> CF_B
- U2 pad 4: VTH_B -> GND
- U2 pad 5: Net-(U6C-+) -> -5V
- U2 pad 6: unconnected-(U2C-NC-Pad6) -> GND
- U2 pad 7: unconnected-(U2C-NC-Pad7) -> /VCO B/SQUARE_B
- U2 pad 8: Net-(U5A--) -> /VCO B/SQUARE_B
- U2 pad 9: GND -> /VCO B/SQUARE_B
- U3 pad 14: Net-(D1C-K) -> /VCO A/SHIFTED_TRI_A
- U3 pad 5: Net-(D1D-K) -> CF_A
- U5 pad 1: Net-(R4-Pad1) -> /VCO A/SQUARE_A
- U5 pad 3: TRIANGLE_B -> TRIANGLE_A
- U5 pad 5: TRIANGLE_A -> TRIANGLE_B
- U5 pad 7: Net-(R5-Pad2) -> /VCO B/SQUARE_B
- U6 pad 14: Net-(D1A-K) -> /VCO B/SHIFTED_TRI_B
- U6 pad 5: Net-(D1B-K) -> CF_B
Routing:
- net +5V: track 43.7 -> 9.12 mm
- net CF_B: track 2.07 -> 35.8 mm, vias 0 -> 1
- net CF_A: track 1.62 -> 32.3 mm, vias 0 -> 2
- net Net-(Q5B-C2): track 0.00 -> 28.9 mm
- net Net-(Q4A-B1): track 0.00 -> 28.0 mm
- net Net-(Q9A-B1): track 0.00 -> 26.5 mm, vias 0 -> 1
- net Net-(D1B-K): track 22.8 -> 0.00 mm, vias 3 -> 0
- net Net-(D1D-K): track 22.2 -> 0.00 mm
- net Net-(Q8B-C2): track 0.00 -> 20.3 mm, vias 0 -> 1
- net Net-(R5-Pad2): track 12.3 -> 0.00 mm, vias 1 -> 0
- net Net-(U3C-+): track 5.94 -> 17.1 mm, vias 0 -> 2
- net Net-(D1A-K): track 11.1 -> 0.00 mm, vias 3 -> 0
- net Net-(U3D--): track 13.7 -> 3.17 mm
- net -5V: track 22.9 -> 12.4 mm, vias 4 -> 3
- net Net-(C2-Pad1): track 10.5 -> 0.00 mm
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- removed copper zone on B.Cu, net +12V
- removed copper zone on B.Cu, net +5V
- removed copper zone on F.Cu, net VTH_A
Other:
- board text added: "REV 1"
- board text removed: "REV 0"
