File: KiCad Files/IO-Power-Tempco.kicad_sch (KiCad schematic)
At the start: 22 parts, among them J1 FLIP PINS, J2 FLIP PINS, U1 DG636E, U10 TLV9032, U2 DG636E, U3 TL074H, U4 AP7370-50FDC, U6 TL074H, U7 TMP6131DECR

Commit message: Updated to Rev 1
Parts:
- C1: renamed from C16; value 0.1u -> 100n
- C11: renamed from C14; value 0.1u -> 100n
- C12: renamed from C15; value 0.1u -> 100n
- C15: renamed from C19; value 0.1u -> 100n
- C16: renamed from C20; value 0.1u -> 100n
- C2: renamed from C1; value 0.1u -> 100n
- C3: renamed from C5; value 0.1u -> 100n
- C5: renamed from C3; value 0.1u -> 100n
- C6: value 0.1u -> 100n
- C8: renamed from C7; value 0.1u -> 100n
- C9: renamed from C8; value 0.1u -> 100n
- R23: renamed from R22; footprint Resistor_SMD:R_0402_1005Metric -> Resistor_SMD:R_0201_0603Metric; Distributor PN C852496 -> C910595; Mfg PN RT0402BRD0711K8L -> AC0201FR-0711K8L; Package 0402 -> 0201; Rating 0.0625W -> 0.05W; Substitute part okay? No -> Yes; Tolerance 0.1% -> 1%
- U1, U2: value DG636E -> DG4053E; symbol DG636E:DG636E -> DG4053E:DG4053E; Distributor LCSC -> Mouser; Distributor PN C458808 -> 78-DG4053EEN-T1-GE4; Mfg PN DG636EEN-T1-GE4 -> DG4053EEN-T1-GE4
- U3, U6: Distributor Digikey -> Mouser; Distributor PN 296-TL074HIDYYRCT-ND -> 595-TL074HIDYYR
- U4: Distributor Digikey -> Mouser; Distributor PN 31-AP7370-50FDC-7CT-ND -> 621-AP7370-50FDC-7
- U5: renamed from U10; Distributor Digikey -> Mouser; Distributor PN 296-TLV9032DSGRCT-ND -> 595-TLV9032DSGR
- U7: Distributor Digikey -> LCSC; Distributor PN 296-TMP6131DECRCT-ND -> C2870682
- renumbered C17 to C13
Connections:
- net +5V: now also U1.14 (V+), U2.14 (V+), U5.8 (V+); no longer U1.1 (EN), U1.11 (V+), U2.1 (EN), U2.11 (V+)
- net -5V: now also U1.5 (V-), U2.5 (V-); no longer U1.2 (V-), U2.2 (V-)
- net GND: now also U1.4 (/EN), U1.6 (GND), U2.4 (/EN), U2.6 (GND), U5.4 (V-), U5.9 (PAD); no longer U1.12 (GND), U2.12 (GND)
- no-connect marks 9 -> 1
Other:
- note added: "TEMP COMPENSATION"
- note removed: "TEMPCO"
