File: KiCad Files/VCO_A.kicad_sch (KiCad schematic)
At the start: 28 parts, among them Q1 DMMT3906W, Q15 DMMT3904W, Q2 MUN5314DW1, Q3 DMMT3906W, Q4 DMMT3904W, Q5 DMMT3906W, Q6 DMMT3904W, Q7 DMMT3906W, U1 DG636E, U3 TL074H, U5 TLV9032

Commit message: Updated to Rev 1
Parts:
- removed C12, C13: 0.01u, Capacitor_SMD:C_0201_0603Metric, symbol Device:C
- removed D1: BAW56DW, Package_TO_SOT_SMD:SOT-363_SC-70-6, symbol Diode:BAW56DW
- removed Q1, Q3: DMMT3906W, Package_TO_SOT_SMD:SOT-363_SC-70-6, symbol DMMT3904W:DMMT3906W
- removed R17: 0, Resistor_SMD:R_0201_0603Metric, symbol Device:R_US
- added R1: 432K, Resistor_SMD:R_0201_0603Metric, symbol Device:R_US
- added R15: 3.32k, Resistor_SMD:R_0201_0603Metric, symbol Device:R_US
- added unit 3 of U1
- C10: renamed from C9; value 100p -> 680p; Distributor PN C408131 -> C161490; Mfg PN GRM033R61E101KA01D -> GRM033R71E681KA01D
- C4: value 0.001u -> 680p; Distributor PN C76943 -> C161490; Mfg PN GRM033R71E102KA01D -> GRM033R71E681KA01D
- R14: renamed from R5; Distributor PN C18164336 -> C473528; Mfg FOJAN -> Uniroyal; Mfg PN FRC0201F4991TS -> 0201WMF4991TEE
- R20: renamed from R19; value 1.02Meg -> 432K; Distributor PN C423793 -> C367623; Mfg Uniroyal -> Walsin; Mfg PN 0201WMF1024TEE -> WR02X4323FAL
- R3: renamed from R1; value 422 -> 365; Distributor PN C474224 -> C423558; Mfg PN 0201WMF4220TEE -> 0201WMF3650TEE
- R8: renamed from R12; Distributor PN C18164336 -> C473528; Mfg FOJAN -> Uniroyal; Mfg PN FRC0201F4991TS -> 0201WMF4991TEE
- U1: value DG636E -> DG4053E; symbol DG636E:DG636E -> DG4053E:DG4053E; Distributor LCSC -> Mouser; Distributor PN C458808 -> 78-DG4053EEN-T1-GE4; Mfg PN DG636EEN-T1-GE4 -> DG4053EEN-T1-GE4
- U3: Distributor Digikey -> Mouser; Distributor PN 296-TL074HIDYYRCT-ND -> 595-TL074HIDYYR
- U5: Distributor Digikey -> Mouser; Distributor PN 296-TLV9032DSGRCT-ND -> 595-TLV9032DSGR
- renumbered Q2 to Q1, Q15 to Q11, Q4 to Q2, Q5 to Q3, Q6 to Q4, Q7 to Q5, R7 to R10, R9 to R12, R11 to R17, R21 to R22, R2 to R4, R3 to R5, R14 to R6
Connections:
- net -5V is gone; now on net SHIFTED_TRI_A: Q2.4 (E1), Q2.5 (E2)
- net +12V: now also Q3.4 (E1), Q3.5 (E2)
- net +5V: now also R17.2; no longer R12.2
- net CF_A: now also Q1.6 (C2), Q4.6 (C2), U3.5 (+), U1.3
- net GND: now also R14.2, U1.11, R1.2; no longer U1.9
- net TRIANGLE_A: now also R12.2, U5.3 (+); no longer U5.5 (+)
- net VTH_A: now also U1.15; no longer U1.4
- net at C4.1, R3.2: now also U1.16, R1.1; no longer U1.3
- net at U3.10 (+): now also U1.13; no longer U1.5
- net at Q4.1 (B2), Q4.2 (B1), Q4.3 (C1): now also U1.1; no longer Q5.6 (C2)
- net at R14.1, U3.13 (-): now also R17.1, R15.2; no longer R17.2
- net SHIFTED_TRI_A: now reaches U3.14
- net SHIFTED_TRI_A: now also R15.1; no longer R17.1
- new net: Q5.6 (C2), U1.2
- new net: U1.12, U5.2 (-)
- new net SQUARE_A: U1.7, U1.8, U1.9, U5.1
Other:
- note removed: "HF COMPENSATION"
- moved on the sheet: C4, Q1A, Q1B, Q3A, Q3B, Q5A, Q5B, R14, R17, U1B
