File: KiCad Files/VCO_B.kicad_sch (KiCad schematic)
At the start: 28 parts, among them Q1 DMMT3904W, Q2 DMMT3906W, Q3 DMMT3906W, Q4 DMMT3906W, Q5 DMMT3906W, Q6 DMMT3904W, Q7 DMMT3904W, U10 TLV9032, U2 TL074H, U6 DG636E, U9 DG636E

Commit message: Updated to Rev 1
Parts:
- removed C13, C14: 0.01u, Capacitor_SMD:C_0201_0603Metric, symbol Device:C
- removed D3: BAW56DW, Package_TO_SOT_SMD:SOT-363_SC-70-6, symbol Diode:BAW56DW
- removed Q4, Q5: DMMT3906W, Package_TO_SOT_SMD:SOT-363_SC-70-6, symbol DMMT3904W:DMMT3906W
- removed R10, R9: 10k, Resistor_SMD:R_0201_0603Metric, symbol Device:R_US
- removed R8: 0, Resistor_SMD:R_0201_0603Metric, symbol Device:R_US
- added R16: 4.99k, Resistor_SMD:R_0201_0603Metric, symbol Device:R_US
- added R18: 10k, Resistor_SMD:R_0201_0603Metric, symbol Device:R_US
- added R2: 432K, Resistor_SMD:R_0201_0603Metric, symbol Device:R_US
- added R27: 3.32k, Resistor_SMD:R_0201_0603Metric, symbol Device:R_US
- added unit 3 of U2
- C14: renamed from C12; value 100p -> 680p; Distributor PN C408131 -> C161490; Mfg PN GRM033R61E101KA01D -> GRM033R71E681KA01D
- C7: renamed from C15; value 0.001u -> 680p; Distributor PN C76943 -> C161490; Mfg PN GRM033R71E102KA01D -> GRM033R71E681KA01D
- R11: value 4.99k -> 10k; Distributor PN C18164336 -> C473048; Mfg FOJAN -> Uniroyal; Mfg PN FRC0201F4991TS -> 0201WMF1002TEE
- R21: renamed from R3; value 1.02Meg -> 432K; Distributor PN C423793 -> C367623; Mfg Uniroyal -> Walsin; Mfg PN 0201WMF1024TEE -> WR02X4323FAL
- R24: renamed from R12; value 422 -> 365; Distributor PN C474224 -> C423558; Mfg PN 0201WMF4220TEE -> 0201WMF3650TEE
- R7: renamed from R15; Distributor PN C18164336 -> C473528; Mfg FOJAN -> Uniroyal; Mfg PN FRC0201F4991TS -> 0201WMF4991TEE
- U2: renamed from U6; value DG636E -> DG4053E; symbol DG636E:DG636E -> DG4053E:DG4053E; Distributor LCSC -> Mouser; Distributor PN C458808 -> 78-DG4053EEN-T1-GE4; Mfg PN DG636EEN-T1-GE4 -> DG4053EEN-T1-GE4
- U2: renamed from U9; value DG636E -> DG4053E; symbol DG636E:DG636E -> DG4053E:DG4053E; Distributor LCSC -> Mouser; Distributor PN C458808 -> 78-DG4053EEN-T1-GE4; Mfg PN DG636EEN-T1-GE4 -> DG4053EEN-T1-GE4
- U5: renamed from U10; Distributor Digikey -> Mouser; Distributor PN 296-TLV9032DSGRCT-ND -> 595-TLV9032DSGR
- U6: renamed from U2; Distributor Digikey -> Mouser; Distributor PN 296-TL074HIDYYRCT-ND -> 595-TL074HIDYYR
- renumbered Q1 to Q10, Q2 to Q6, Q3 to Q8, Q6 to Q9, R4 to R19, R17 to R25, R16 to R26, R14 to R9
Connections:
- net +12V: now also Q6.4 (E1), Q6.5 (E2)
- net +5V: now also R18.2; no longer R13.2
- net CF_B: now also Q9.6 (C2), U6.5 (+), U2.3
- net GND: now also R11.2, U2.11, R16.2, R2.2; no longer U2.4
- net SAWTOOTH_B: now also U6.8; no longer U6.14
- net TRIANGLE_B: now also R13.2, U5.5 (+); no longer U5.3 (+)
- net VTH_B: now also U2.10, U2.15; no longer U2.3, U2.4
- net at C7.1, R24.2: now also U2.16, R2.1; no longer U2.3
- net at R13.1: now also R11.1, U6.12 (+); no longer U6.10 (+)
- net at R25.1, R26.2: now also U6.9 (-); no longer U6.13 (-)
- net at Q9.1 (B2), Q9.2 (B1), Q9.3 (C1): now also U2.1; no longer Q8.6 (C2)
- net -5V renamed SHIFTED_TRI_B
- net SHIFTED_TRI_B: now also U6.14, R27.1
- new net: U2.13, U6.10 (+)
- new net: R16.1, R18.1, R27.2, U6.13 (-)
- new net: U2.12, U5.6 (-)
- new net: Q8.6 (C2), U2.2
- new net SQUARE_B: U2.7, U2.8, U2.9, U5.7
Other:
- note removed: "HF COMPENSATION"
- moved on the sheet: C7, Q6A, Q6B, Q8A, Q8B, U2B
